Commit message: Adapting to futurhand format, first pass

File: fanuc_crx_description/urdf/crx10ia_urdf_macro.xacro (robot description, xacro)
@@ -380,5 +380,5 @@
     <joint name="${prefix}child_joint" type="fixed">
       <origin xyz="0 0 0" rpy="0 0 0" />
-      <parent link="${prefix}flange" />
+      <parent link="${prefix}fanuc_flange" />
       <child link="${child}" />
     </joint>
